Commit message: Add colors to the model

File: src/bumperbot_description/urdf/bumperbot.gazebo.xacro (robot description, xacro)
@@ -1,5 +1,10 @@
 <?xml version="1.0"?>
 <robot xmlns:xacro="http://www.ros.org/wiki/xacro" name="bumperbot" >
+    <!-- Gazebo colors for visualization in simulation -->
+    <gazebo reference="base_link">
+        <material>Gazebo/Black</material>
+    </gazebo>
     <gazebo reference="wheel_right_link">
+        <material>Gazebo/Blue</material>
         <mu1>100000000000000.0</mu1>
         <mu2>100000000000000.0</mu2>
@@ -12,4 +17,5 @@
     </gazebo>
     <gazebo reference="wheel_left_link">
+        <material>Gazebo/Blue</material>
         <mu1>100000000000000.0</mu1>
         <mu2>100000000000000.0</mu2>
@@ -22,4 +28,5 @@
     </gazebo>
     <gazebo reference="caster_front_link">
+        <material>Gazebo/Grey</material>
         <mu1>0.1</mu1>
         <mu2>0.1</mu2>
@@ -31,4 +38,5 @@
     </gazebo>
     <gazebo reference="caster_rear_link">
+        <material>Gazebo/Grey</material>
         <mu1>0.1</mu1>
         <mu2>0.1</mu2>
@@ -38,4 +46,7 @@
         <minDepth>0.001</minDepth>
         <maxVel>0.01</maxVel>
+    </gazebo>
+    <gazebo reference="can_link">
+        <material>Gazebo/Red</material>
     </gazebo>
     <gazebo>

File: src/bumperbot_description/urdf/bumperbot.urdf.xacro (robot description, xacro)
@@ -3,4 +3,23 @@
     <!-- This argument is used to determine if we are using ros 2 humble (true) or jazzy (false)-->
     <xacro:arg name="is_ignition" default="true"/>
+    <!-- Define materials/colors -->
+    <material name="blue">
+        <color rgba="0.2 0.2 0.8 1.0"/>
+    </material>
+    <material name="black">
+        <color rgba="0.1 0.1 0.1 1.0"/>
+    </material>
+    <material name="white">
+        <color rgba="1.0 1.0 1.0 1.0"/>
+    </material>
+    <material name="grey">
+        <color rgba="0.5 0.5 0.5 1.0"/>
+    </material>
+    <material name="red">
+        <color rgba="0.8 0.0 0.0 1.0"/>
+    </material>
+    <material name="silver">
+        <color rgba="0.75 0.75 0.75 1.0"/>
+    </material>
     <!-- Include another model-->
     <xacro:include filename="$(find bumperbot_description)/urdf/bumperbot.gazebo.xacro" />
@@ -20,4 +39,5 @@
                 <mesh filename="package://bumperbot_description/meshes/base_link.STL"  />
            </geometry>
+           <material name="black"/>
         </visual>
         <!-- This parameters are required for gazebo -->
@@ -45,4 +65,5 @@
                 <mesh filename = "package://bumperbot_description/meshes/wheel_right_link.STL"></mesh>
             </geometry>
+            <material name="blue"/>
         </visual>
         <collision>
@@ -71,4 +92,5 @@
                 <mesh filename = "package://bumperbot_description/meshes/wheel_left_link.STL"></mesh>
             </geometry>
+            <material name="blue"/>
         </visual>
         <collision>
@@ -97,4 +119,5 @@
                 <mesh filename = "package://bumperbot_description/meshes/caster_front_link.STL"></mesh>
             </geometry>
+            <material name="grey"/>
         </visual>
         <collision>
@@ -122,4 +145,5 @@
                 <mesh filename = "package://bumperbot_description/meshes/caster_rear_link.STL"></mesh>
             </geometry>
+            <material name="grey"/>
         </visual>
         <collision>
@@ -142,4 +166,5 @@
                 <mesh filename= "package://bumperbot_description/meshes/can.STL"></mesh>
             </geometry>
+            <material name="red"/>
         </visual>
     </link>
